Commit message: Rotated IMU in realsense to line up with real

File: ifo_description/urdf/realsense_d435i.xacro (robot description, xacro)
@@ -36,4 +36,85 @@
     <child link="${name}_link"/>
   </joint>
+  <link name="${name}_imu_link"/>
+  <joint name="${name}_imu_joint" type="fixed">
+      <!-- Rotate and translate IMU to be same as real realsense-->
+      <!-- Frame is y DOWN, z forward-->
+    <origin xyz="-0.0051 0.01195 -0.01174" rpy="-1.5707 0 -1.5707" />
+    <parent link="${name}_link"/>
+    <child link="${name}_imu_link"/>
+  </joint>
+  <!-- =================================================================== -->
+  <!--                                 IMU                                 -->
+  <!-- =================================================================== -->
+  <gazebo reference="${name}_imu_link">
+    <sensor name="imu_sensor" type="imu">
+      <always_on>1</always_on>
+      <update_rate>100.0</update_rate>
+      <topic>${name}/imu</topic>
+      <imu>
+        <angular_velocity>
+          <x>
+            <noise type="gaussian">
+              <mean>0.0</mean>
+              <stddev>0.01</stddev>
+              <bias_mean>0.0</bias_mean>
+              <bias_stddev>0.0001</bias_stddev>
+            </noise>
+          </x>
+          <y>
+            <noise type="gaussian">
+              <mean>0.0</mean>
+              <stddev>0.01</stddev>
+              <bias_mean>0.0</bias_mean>
+              <bias_stddev>0.0001</bias_stddev>
+            </noise>
+          </y>
+          <z>
+            <noise type="gaussian">
+              <mean>0.0</mean>
+              <stddev>0.01</stddev>
+              <bias_mean>0.0</bias_mean>
+              <bias_stddev>0.0001</bias_stddev>
+            </noise>
+          </z>
+        </angular_velocity>
+        <linear_acceleration>
+          <x>
+            <noise type="gaussian">
+              <mean>0.0</mean>
+              <stddev>0.01</stddev>
+              <bias_mean>0.0</bias_mean>
+              <bias_stddev>0.0001</bias_stddev>
+            </noise>
+          </x>
+          <y>
+            <noise type="gaussian">
+              <mean>0.0</mean>
+              <stddev>0.01</stddev>
+              <bias_mean>0.0</bias_mean>
+              <bias_stddev>0.0001</bias_stddev>
+            </noise>
+          </y>
+          <z>
+            <noise type="gaussian">
+              <mean>0.0</mean>
+              <stddev>0.01</stddev>
+              <bias_mean>0.0</bias_mean>
+              <bias_stddev>0.0001</bias_stddev>
+            </noise>
+          </z>
+        </linear_acceleration>
+      </imu>
+      <plugin filename="libgazebo_ros_imu_sensor.so" name="imu_plugin">
+        <robotNamespace></robotNamespace>
+        <topicName>${name}/imu</topicName>
+        <bodyName>${name}_link</bodyName>
+        <updateRateHZ>100.0</updateRateHZ>
+        <xyzOffset>0 0 0</xyzOffset>
+        <rpyOffset>0 0 0</rpyOffset>
+        <frameName>${name}_link</frameName>
+      </plugin>
+    </sensor>
+  </gazebo>
   <gazebo reference="${name}_link">
     <self_collide>0</self_collide>
@@ -43,5 +124,5 @@
       <cast_shadows>1</cast_shadows>
     </visual>
-    <inertial>
+    <!-- <inertial>
       <mass> 0.0000001 </mass>
       <inertia>
@@ -50,79 +131,5 @@
         <izz> 1e-10 </izz>
       </inertia>
-    </inertial>
-    <!-- =================================================================== -->
-    <!--                                 IMU                                 -->
-    <!-- =================================================================== -->
-    <sensor name="imu_sensor" type="imu">
-      <!-- Rotate and translate IMU to be same as real realsense-->
-      <!-- Frame is y up, z forward-->
-      <pose>-0.0051 0.01195 -0.01174 -1.5707 0 -1.5707</pose>
-      <always_on>1</always_on>
-      <update_rate>100.0</update_rate>
-      <topic>${name}/imu</topic>
-      <imu>
-        <angular_velocity>
-          <x>
-            <noise type="gaussian">
-              <mean>0.0</mean>
-              <stddev>0.01</stddev>
-              <bias_mean>0.0</bias_mean>
-              <bias_stddev>0.0001</bias_stddev>
-            </noise>
-          </x>
-          <y>
-            <noise type="gaussian">
-              <mean>0.0</mean>
-              <stddev>0.01</stddev>
-              <bias_mean>0.0</bias_mean>
-              <bias_stddev>0.0001</bias_stddev>
-            </noise>
-          </y>
-          <z>
-            <noise type="gaussian">
-              <mean>0.0</mean>
-              <stddev>0.01</stddev>
-              <bias_mean>0.0</bias_mean>
-              <bias_stddev>0.0001</bias_stddev>
-            </noise>
-          </z>
-        </angular_velocity>
-        <linear_acceleration>
-          <x>
-            <noise type="gaussian">
-              <mean>0.0</mean>
-              <stddev>0.01</stddev>
-              <bias_mean>0.0</bias_mean>
-              <bias_stddev>0.0001</bias_stddev>
-            </noise>
-          </x>
-          <y>
-            <noise type="gaussian">
-              <mean>0.0</mean>
-              <stddev>0.01</stddev>
-              <bias_mean>0.0</bias_mean>
-              <bias_stddev>0.0001</bias_stddev>
-            </noise>
-          </y>
-          <z>
-            <noise type="gaussian">
-              <mean>0.0</mean>
-              <stddev>0.01</stddev>
-              <bias_mean>0.0</bias_mean>
-              <bias_stddev>0.0001</bias_stddev>
-            </noise>
-          </z>
-        </linear_acceleration>
-      </imu>
-      <plugin filename="libgazebo_ros_imu_sensor.so" name="imu_plugin">
-        <robotNamespace></robotNamespace>
-        <topicName>${name}/imu</topicName>
-        <bodyName>${name}_link</bodyName>
-        <updateRateHZ>200.0</updateRateHZ>
-        <xyzOffset>0 0 0</xyzOffset>
-        <rpyOffset>0 0 0</rpyOffset>
-        <frameName>${name}_link</frameName>
-      </plugin>
-    </sensor>
+    </inertial> -->
     <!-- =================================================================== -->
     <!--                              CAMERAS                                -->

Commit message: Fixed realsense camera locations

File: ifo_description/urdf/realsense_d435i.xacro (robot description, xacro)
@@ -36,4 +36,7 @@
     <child link="${name}_link"/>
   </joint>
+  <!-- =================================================================== -->
+  <!--                                 IMU                                 -->
+  <!-- =================================================================== -->
   <link name="${name}_imu_link"/>
   <joint name="${name}_imu_joint" type="fixed">
@@ -44,7 +47,4 @@
     <child link="${name}_imu_link"/>
   </joint>
-  <!-- =================================================================== -->
-  <!--                                 IMU                                 -->
-  <!-- =================================================================== -->
   <gazebo reference="${name}_imu_link">
     <sensor name="imu_sensor" type="imu">
@@ -117,5 +117,19 @@
     </sensor>
   </gazebo>
-  <gazebo reference="${name}_link">
+  <!-- =================================================================== -->
+  <!--                              CAMERAS                                -->
+  <!-- =================================================================== -->
+  <!--
+  See the following link for dimensions. Page 88.
+  https://www.intelrealsense.com/wp-content/uploads/2022/03/Intel-RealSense-D400-Series-Datasheet-March-2022.pdf
+  -->
+  <!-- _____________________ Realsense colour camera ______________________-->
+  <link name="${name}_color_link"/>
+  <joint name="${name}_color_joint" type="fixed">
+    <origin xyz="0 0.0325 0" rpy="0 0 0" />
+    <parent link="${name}_link"/>
+    <child link="${name}_color_link"/>
+  </joint>
+  <gazebo reference="${name}_color_link">
     <self_collide>0</self_collide>
     <kinematic>0</kinematic>
@@ -124,18 +138,6 @@
       <cast_shadows>1</cast_shadows>
     </visual>
-    <!-- <inertial>
-      <mass> 0.0000001 </mass>
-      <inertia>
-        <ixx> 1e-10 </ixx>
-        <iyy> 1e-10 </iyy>
-        <izz> 1e-10 </izz>
-      </inertia>
-    </inertial> -->
-    <!-- =================================================================== -->
-    <!--                              CAMERAS                                -->
-    <!-- =================================================================== -->
-    <!-- Realsense colour camera-->
     <sensor name="${name}_color" type="camera">
-      <pose>0 -0.0115 0 0 0 0</pose>
+      <!-- <pose>0 -0.0115 0 0 0 0</pose> -->
       <camera name="${name}">
         <horizontal_fov>1.211259</horizontal_fov>
@@ -159,7 +161,21 @@
       <visualize>0</visualize>
     </sensor>
-    <!-- Realsense infrared camera 1 (left)-->
+  </gazebo>
+  <!-- _______________ Realsense infrared camera 1 (left) _________________-->
+  <link name="${name}_infra1_link"/>
+  <joint name="${name}_infra1_joint" type="fixed">
+    <origin xyz="0 0.0175 0" rpy="0 0 0" />
+    <parent link="${name}_link"/>
+    <child link="${name}_infra1_link"/>
+  </joint>
+  <gazebo reference="${name}_infra1_link">
+    <self_collide>0</self_collide>
+    <kinematic>0</kinematic>
+    <gravity>0</gravity>
+    <visual>
+      <cast_shadows>1</cast_shadows>
+    </visual>
     <sensor name="${name}_ired1" type="camera">
-      <pose>0 0.0175 0 0 0 0</pose>
+      <!-- <pose>0 0.0175 0 0 0 0</pose> -->
       <camera name="${name}">
         <horizontal_fov>1.487021</horizontal_fov>
@@ -183,7 +199,21 @@
       <visualize>0</visualize>
     </sensor>
-    <!-- Realsense infrared camera 2 (right)-->
+  </gazebo>
+  <!-- _______________ Realsense infrared camera 2 (right) ________________-->
+  <link name="${name}_infra2_link"/>
+  <joint name="${name}_infra2_joint" type="fixed">
+    <origin xyz="0 -0.0325 0" rpy="0 0 0" />
+    <parent link="${name}_link"/>
+    <child link="${name}_infra2_link"/>
+  </joint>
+  <gazebo reference="${name}_infra2_link">
+    <self_collide>0</self_collide>
+    <kinematic>0</kinematic>
+    <gravity>0</gravity>
+    <visual>
+      <cast_shadows>1</cast_shadows>
+    </visual>
     <sensor name="${name}_ired2" type="camera">
-      <pose>0 -0.0325 0 0 0 0</pose>
+      <!-- <pose>0 -0.0325 0 0 0 0</pose> -->
       <camera name="${name}">
         <horizontal_fov>1.487021</horizontal_fov>
@@ -207,7 +237,21 @@
       <visualize>0</visualize>
     </sensor>
-    <!-- Realsense depth camera-->
+  </gazebo>
+  <!-- _____________________ Realsense depth camera  ______________________-->
+  <link name="${name}_depth_link"/>
+  <joint name="${name}_depth_joint" type="fixed">
+    <origin xyz="0 0.0325 0" rpy="0 0 0" />
+    <parent link="${name}_link"/>
+    <child link="${name}_depth_link"/>
+  </joint>
+  <gazebo reference="${name}_depth_link">
+    <self_collide>0</self_collide>
+    <kinematic>0</kinematic>
+    <gravity>0</gravity>
+    <visual>
+      <cast_shadows>1</cast_shadows>
+    </visual>
     <sensor name="${name}_depth" type="depth">
-    <pose>0 0.0325 0 0 0 0</pose>
+    <!-- <pose>0 0.0325 0 0 0 0</pose> -->
       <camera name="${name}">
         <horizontal_fov>1.487021</horizontal_fov>
@@ -231,33 +275,33 @@
     </sensor>
   </gazebo>
+  <!-- ________________________ Realsense PLUGIN  _________________________-->
   <gazebo>
-  <!-- Realsense Plugin -->
-  <plugin name="/${name}" filename="librealsense_gazebo_plugin.so">
-    <prefix>${name}_</prefix>
-    <!-- Color camera settings-->
-    <colorUpdateRate>15.0</colorUpdateRate>
-    <colorTopicName>color/image_raw</colorTopicName>
-    <colorCameraInfoTopicName>color/camera_info</colorCameraInfoTopicName>
-    <colorOpticalframeName>${name}_color_optical_frame</colorOpticalframeName>
-    <!-- Infrared camera settings-->
-    <infraredUpdateRate>15.0</infraredUpdateRate>
-    <infrared1TopicName>infra1/image_raw</infrared1TopicName>
-    <infrared1CameraInfoTopicName>infra1/camera_info</infrared1CameraInfoTopicName>
-    <infrared1OpticalframeName>${name}_infrared1_optical_frame</infrared1OpticalframeName>
-    <infrared2TopicName>infra2/image_raw</infrared2TopicName>
-    <infrared2CameraInfoTopicName>infra2/camera_info</infrared2CameraInfoTopicName>
-    <infrared2OpticalframeName>${name}_infrared2_optical_frame</infrared2OpticalframeName>
-    <!-- Depth camera settings-->
-    <depthUpdateRate>15.0</depthUpdateRate>
-    <depthTopicName>depth/image_raw</depthTopicName>
-    <depthCameraInfoTopicName>depth/camera_info</depthCameraInfoTopicName>
-    <depthOpticalframeName>${name}_depth_optical_frame</depthOpticalframeName>
-    <rangeMinDepth>0.1</rangeMinDepth>
-    <rangeMaxDepth>10.0</rangeMaxDepth>
-    <pointCloud>true</pointCloud>
-    <pointCloudTopicName>depth/color/points</pointCloudTopicName>
-    <pointCloudCutoff>0.25</pointCloudCutoff>
-    <pointCloudCutoffMax>9.0</pointCloudCutoffMax>
-  </plugin>
+    <plugin name="/${name}" filename="librealsense_gazebo_plugin.so">
+      <prefix>${name}_</prefix>
+      <!-- Color camera settings-->
+      <colorUpdateRate>15.0</colorUpdateRate>
+      <colorTopicName>color/image_raw</colorTopicName>
+      <colorCameraInfoTopicName>color/camera_info</colorCameraInfoTopicName>
+      <colorOpticalframeName>${name}_color_optical_frame</colorOpticalframeName>
+      <!-- Infrared camera settings-->
+      <infraredUpdateRate>15.0</infraredUpdateRate>
+      <infrared1TopicName>infra1/image_raw</infrared1TopicName>
+      <infrared1CameraInfoTopicName>infra1/camera_info</infrared1CameraInfoTopicName>
+      <infrared1OpticalframeName>${name}_infrared1_optical_frame</infrared1OpticalframeName>
+      <infrared2TopicName>infra2/image_raw</infrared2TopicName>
+      <infrared2CameraInfoTopicName>infra2/camera_info</infrared2CameraInfoTopicName>
+      <infrared2OpticalframeName>${name}_infrared2_optical_frame</infrared2OpticalframeName>
+      <!-- Depth camera settings-->
+      <depthUpdateRate>15.0</depthUpdateRate>
+      <depthTopicName>depth/image_raw</depthTopicName>
+      <depthCameraInfoTopicName>depth/camera_info</depthCameraInfoTopicName>
+      <depthOpticalframeName>${name}_depth_optical_frame</depthOpticalframeName>
+      <rangeMinDepth>0.1</rangeMinDepth>
+      <rangeMaxDepth>10.0</rangeMaxDepth>
+      <pointCloud>true</pointCloud>
+      <pointCloudTopicName>depth/color/points</pointCloudTopicName>
+      <pointCloudCutoff>0.25</pointCloudCutoff>
+      <pointCloudCutoffMax>9.0</pointCloudCutoffMax>
+    </plugin>
   </gazebo>
 </xacro:macro>
