Commit message: Added realsense in new URDF model

File: ifo_description/urdf/ifo.xacro (robot description, xacro)
@@ -6,3 +6,8 @@
     <xacro:include filename="$(find ifo_description)/urdf/ifo_base.xacro" />
     <xacro:ifo_base_macro mavlink_tcp_port="$(arg mavlink_tcp_port)" mavlink_udp_port="$(arg mavlink_udp_port)"/>
+    <!-- Include realsense -->
+    <xacro:include filename="$(find realsense_gazebo_description)/urdf/_d435i.urdf.xacro"/>
+    <xacro:sensor_d435i parent="base_link">
+        <origin xyz="0.10 0 0" rpy="0 0 0" />
+    </xacro:sensor_d435i>
 </robot>

Commit message: Fixed realsense IMU problem by making simplified version

File: ifo_description/urdf/ifo.xacro (robot description, xacro)
@@ -8,11 +8,6 @@
     <xacro:ifo_base_macro mavlink_tcp_port="$(arg mavlink_tcp_port)" mavlink_udp_port="$(arg mavlink_udp_port)"/>
     <!-- Include realsense -->
-    <xacro:include filename="$(find realsense_gazebo_description)/urdf/_d435i.urdf.xacro"/>
-    <xacro:sensor_d435i
-            name="$(arg namespace)/realsense"
-            topics_ns="$(arg namespace)/realsense"
-            parent="base_link" accel_fps="200" gyro_fps="200"
-            unite_imu_method="copy">
-        <origin xyz="0.10 0 0" rpy="0 0 0" />
-    </xacro:sensor_d435i>
+    <xacro:include filename="$(find ifo_description)/urdf/realsense_d435i.xacro"/>
+    <xacro:realsense_d435i>
+    </xacro:realsense_d435i>
 </robot>

Commit message: Completely removed old SDF models

File: ifo_description/urdf/ifo.xacro (robot description, xacro)
@@ -9,5 +9,6 @@
     <!-- Include realsense -->
     <xacro:include filename="$(find ifo_description)/urdf/realsense_d435i.xacro"/>
-    <xacro:realsense_d435i>
+    <xacro:realsense_d435i parent="base_link" name="camera">
+        <origin xyz="0.12 0 0" rpy="0 0 0" />
     </xacro:realsense_d435i>
 </robot>

File: ifo_description/urdf/ifo_base.xacro (robot description, xacro)
@@ -116,5 +116,5 @@
             <mesh>
               <scale>1 1 1</scale>
-              <uri>model://ifo_base/meshes/iris_prop_ccw.dae</uri>
+              <uri>$(find ifo_description)/meshes/iris_prop_ccw.dae</uri>
             </mesh>
           </geometry>
@@ -203,5 +203,5 @@
             <mesh>
               <scale>1 1 1</scale>
-              <uri>model://ifo_base/meshes/iris_prop_ccw.dae</uri>
+              <uri>$(find ifo_description)/meshes/iris_prop_ccw.dae</uri>
             </mesh>
           </geometry>
@@ -290,5 +290,5 @@
             <mesh>
               <scale>1 1 1</scale>
-              <uri>model://ifo_base/meshes/iris_prop_cw.dae</uri>
+              <uri>$(find ifo_description)/meshes/iris_prop_cw.dae</uri>
             </mesh>
           </geometry>
@@ -377,5 +377,5 @@
             <mesh>
               <scale>1 1 1</scale>
-              <uri>model://ifo_base/meshes/iris_prop_cw.dae</uri>
+              <uri>$(find ifo_description)/meshes/iris_prop_cw.dae</uri>
             </mesh>
           </geometry>

File: ifo_description/urdf/realsense_d435i.xacro (robot description, xacro)
@@ -1,20 +1,22 @@
 <?xml version="1.0"?>
 <robot xmlns:xacro="http://www.ros.org/wiki/xacro">
-<xacro:macro name="realsense_d435i">
-  <link name="camera_link">
+<xacro:macro name="realsense_d435i" params="parent
+                                            *origin
+                                            name:=camera">
+  <link name="${name}_link">
     <!-- Visual rendering-->
     <visual>
       <origin xyz="0 0 0" rpy="1.5707 0 1.5707" />
       <geometry>
-        <mesh filename="package://ifo_description/meshes/d435.dae" />
+        <mesh filename="$(find ifo_description)/meshes/d435.dae" />
       </geometry>
     </visual>
   </link>
-  <joint name="camera_joint" type="fixed">
-    <origin xyz="0.12 0 0" rpy="0 0 0" />
-    <parent link="base_link"/>
-    <child link="camera_link"/>
+  <joint name="${name}_joint" type="fixed">
+    <xacro:insert_block name="origin"/>
+    <parent link="${parent}"/>
+    <child link="${name}_link"/>
   </joint>
-  <gazebo reference="camera_link">
+  <gazebo reference="${name}_link">
     <self_collide>0</self_collide>
     <kinematic>0</kinematic>
@@ -40,5 +42,5 @@
       <always_on>1</always_on>
       <update_rate>100.0</update_rate>
-      <topic>/camera/imu</topic>
+      <topic>${name}/imu</topic>
       <imu>
         <angular_velocity>
@@ -97,10 +99,10 @@
       <plugin filename="libgazebo_ros_imu_sensor.so" name="imu_plugin">
         <robotNamespace></robotNamespace>
-        <topicName>camera/imu</topicName>
-        <bodyName>camera_link</bodyName>
+        <topicName>${name}/imu</topicName>
+        <bodyName>${name}_link</bodyName>
         <updateRateHZ>200.0</updateRateHZ>
         <xyzOffset>0 0 0</xyzOffset>
         <rpyOffset>0 0 0</rpyOffset>
-        <frameName>camera_link</frameName>
+        <frameName>${name}_link</frameName>
       </plugin>
     </sensor>
@@ -109,7 +111,7 @@
     <!-- =================================================================== -->
     <!-- Realsense colour camera-->
-    <sensor name="camera_color" type="camera">
+    <sensor name="${name}_color" type="camera">
       <pose>0 -0.0115 0 0 0 0</pose>
-      <camera name="camera">
+      <camera name="${name}">
         <horizontal_fov>1.211259</horizontal_fov>
         <image>
@@ -133,7 +135,7 @@
     </sensor>
     <!-- Realsense infrared camera 1 (left)-->
-    <sensor name="camera_ired1" type="camera">
+    <sensor name="${name}_ired1" type="camera">
       <pose>0 0.0175 0 0 0 0</pose>
-      <camera name="camera">
+      <camera name="${name}">
         <horizontal_fov>1.487021</horizontal_fov>
         <image>
@@ -157,7 +159,7 @@
     </sensor>
     <!-- Realsense infrared camera 2 (right)-->
-    <sensor name="camera_ired2" type="camera">
+    <sensor name="${name}_ired2" type="camera">
       <pose>0 -0.0325 0 0 0 0</pose>
-      <camera name="camera">
+      <camera name="${name}">
         <horizontal_fov>1.487021</horizontal_fov>
         <image>
@@ -181,7 +183,7 @@
     </sensor>
     <!-- Realsense depth camera-->
-    <sensor name="camera_depth" type="depth">
+    <sensor name="${name}_depth" type="depth">
     <pose>0 0.0325 0 0 0 0</pose>
-      <camera name="camera">
+      <camera name="${name}">
         <horizontal_fov>1.487021</horizontal_fov>
         <image>
@@ -206,24 +208,24 @@
   <gazebo>
   <!-- Realsense Plugin -->
-  <plugin name="/camera" filename="librealsense_gazebo_plugin.so">
-    <prefix>camera_</prefix>
+  <plugin name="/${name}" filename="librealsense_gazebo_plugin.so">
+    <prefix>${name}_</prefix>
     <!-- Color camera settings-->
     <colorUpdateRate>15.0</colorUpdateRate>
     <colorTopicName>color/image_raw</colorTopicName>
     <colorCameraInfoTopicName>color/camera_info</colorCameraInfoTopicName>
-    <colorOpticalframeName>camera_color_optical_frame</colorOpticalframeName>
+    <colorOpticalframeName>${name}_color_optical_frame</colorOpticalframeName>
     <!-- Infrared camera settings-->
     <infraredUpdateRate>15.0</infraredUpdateRate>
     <infrared1TopicName>infra1/image_raw</infrared1TopicName>
     <infrared1CameraInfoTopicName>infra1/camera_info</infrared1CameraInfoTopicName>
-    <infrared1OpticalframeName>camera_infrared1_optical_frame</infrared1OpticalframeName>
+    <infrared1OpticalframeName>${name}_infrared1_optical_frame</infrared1OpticalframeName>
     <infrared2TopicName>infra2/image_raw</infrared2TopicName>
     <infrared2CameraInfoTopicName>infra2/camera_info</infrared2CameraInfoTopicName>
-    <infrared2OpticalframeName>camera_infrared2_optical_frame</infrared2OpticalframeName>
+    <infrared2OpticalframeName>${name}_infrared2_optical_frame</infrared2OpticalframeName>
     <!-- Depth camera settings-->
     <depthUpdateRate>15.0</depthUpdateRate>
     <depthTopicName>depth/image_raw</depthTopicName>
     <depthCameraInfoTopicName>depth/camera_info</depthCameraInfoTopicName>
-    <depthOpticalframeName>camera_depth_optical_frame</depthOpticalframeName>
+    <depthOpticalframeName>${name}_depth_optical_frame</depthOpticalframeName>
     <rangeMinDepth>0.1</rangeMinDepth>
     <rangeMaxDepth>10.0</rangeMaxDepth>

Commit message: Realsense now work properly with multi agents. Tested with flying and VINS-Fusion.

File: ifo_description/urdf/ifo.xacro (robot description, xacro)
@@ -9,5 +9,5 @@
     <!-- Include realsense -->
     <xacro:include filename="$(find ifo_description)/urdf/realsense_d435i.xacro"/>
-    <xacro:realsense_d435i parent="base_link" name="camera">
+    <xacro:realsense_d435i parent="base_link" name="$(arg namespace)/camera">
         <origin xyz="0.12 0 0" rpy="0 0 0" />
     </xacro:realsense_d435i>

File: ifo_description/urdf/realsense_d435i.xacro (robot description, xacro)
@@ -4,4 +4,22 @@
                                             *origin
                                             name:=camera">
+  <!-- Realsense D435i macro
+    Calling this macro from a top-level xacro file will include an Intel
+    Realsense D435i camera, publishing IMU readings as well as color,
+    2 x infrared, and depth image topics.
+    Usage (in a top-level xacro file)
+    <xacro:include filename="path/to/realsense_d435i.xacro"/>
+    <xacro:realsense_d435i parent="base_link" name="$(arg namespace)/camera">
+        <origin xyz="0.12 0 0" rpy="0 0 0" />
+    </xacro:realsense_d435i>
+    Note that multiple cameras can coexist in a simulation by giving each camera
+    a unique name.
+    TODO
+    - Parameterize everything using params
+    To understand this file you should really look at the URDF tutorials:
+    https://wiki.ros.org/urdf/Tutorials
+    In addition to how to use URDF with Gazebo
+    http://gazebosim.org/tutorials/?tut=ros_urdf
+    -->
   <link name="${name}_link">
     <!-- Visual rendering-->

Commit message: added argument to add/omit realsense simulation

File: ifo_description/urdf/ifo.xacro (robot description, xacro)
@@ -2,15 +2,17 @@
 <robot name='ifo' xmlns:xacro="http://www.ros.org/wiki/xacro">
     <!-- This is the main top-level file-->
-    <!-- TODO: add user option to omit realsense for a "lighter" version. -->
     <xacro:arg name="mavlink_tcp_port" default="4560" />
     <xacro:arg name="mavlink_udp_port" default="14560" />
     <xacro:arg name="namespace" default=""/>
+    <xacro:arg name="camera" default="true"/>
     <!-- Include base -->
     <xacro:include filename="$(find ifo_description)/urdf/ifo_base.xacro" />
     <xacro:ifo_base_macro mavlink_tcp_port="$(arg mavlink_tcp_port)" mavlink_udp_port="$(arg mavlink_udp_port)"/>
     <!-- Include realsense -->
-    <xacro:include filename="$(find ifo_description)/urdf/realsense_d435i.xacro"/>
-    <xacro:realsense_d435i parent="base_link" name="$(arg namespace)/camera">
-        <origin xyz="0.12 0 0" rpy="0 0 0" />
-    </xacro:realsense_d435i>
+    <xacro:if value="$(arg camera)">
+        <xacro:include filename="$(find ifo_description)/urdf/realsense_d435i.xacro"/>
+        <xacro:realsense_d435i parent="base_link" name="$(arg namespace)/camera">
+            <origin xyz="0.12 0 0" rpy="0 0 0" />
+        </xacro:realsense_d435i>
+    </xacro:if>
 </robot>
